Commit message: rover update

File: asd_robot/urdf/leo_rover.gazebo.xacro (robot description, xacro)
@@ -9,11 +9,10 @@
   </gazebo>
   <gazebo reference="wheel_FL_link">
-    <mu1>3.0</mu1>
-    <mu2>3.0</mu2>
-    <kp>500000.0</kp>
-    <kd>10.0</kd>
-    <minDepth>0.001</minDepth>
-    <maxVel>5.0</maxVel>
+    <kp>1e6</kp>
+    <kd>1.0</kd>
+    <mu1>5.0</mu1>
+    <mu2>0.5</mu2>
     <fdir1>1 0 0</fdir1>
+    <minDepth>0.003</minDepth>
   </gazebo>
   <gazebo reference="wheel_FL_joint">
@@ -28,11 +27,10 @@
   </gazebo>
   <gazebo reference="wheel_RL_link">
-    <mu1>3.0</mu1>
-    <mu2>3.0</mu2>
-    <kp>500000.0</kp>
-    <kd>10.0</kd>
-    <minDepth>0.001</minDepth>
-    <maxVel>6.0</maxVel>
+    <kp>1e6</kp>
+    <kd>1.0</kd>
+    <mu1>5.0</mu1>
+    <mu2>0.5</mu2>
     <fdir1>1 0 0</fdir1>
+    <minDepth>0.003</minDepth>
   </gazebo>
   <gazebo reference="wheel_RL_joint">
@@ -47,11 +45,10 @@
   </gazebo>
   <gazebo reference="wheel_FR_link">
-    <mu1>3.0</mu1>
-    <mu2>3.0</mu2>
-    <kp>500000.0</kp>
-    <kd>10.0</kd>
-    <minDepth>0.001</minDepth>
-    <maxVel>6.0</maxVel>
+    <kp>1e6</kp>
+    <kd>1.0</kd>
+    <mu1>5.0</mu1>
+    <mu2>0.5</mu2>
     <fdir1>1 0 0</fdir1>
+    <minDepth>0.003</minDepth>
   </gazebo>
   <gazebo reference="wheel_FR_joint">
@@ -66,11 +63,10 @@
   </gazebo>
   <gazebo reference="wheel_RR_link">
-    <mu1>3.0</mu1>
-    <mu2>3.0</mu2>
-    <kp>500000.0</kp>
-    <kd>10.0</kd>
-    <minDepth>0.001</minDepth>
-    <maxVel>6.0</maxVel>
+    <kp>1e6</kp>
+    <kd>1.0</kd>
+    <mu1>5.0</mu1>
+    <mu2>0.5</mu2>
     <fdir1>1 0 0</fdir1>
+    <minDepth>0.003</minDepth>
   </gazebo>
   <gazebo reference="wheel_RR_joint">

File: asd_robot/urdf/leo_rover.urdf.xacro (robot description, xacro)
@@ -93,6 +93,6 @@
     <child link="rocker_L_link"/>
     <axis xyz="0 1 0"/>
-    <limit effort="10" lower="-0.24" upper="0.24" velocity="0.5"/>
-    <dynamics friction="0.1" damping="0.1"/>
+    <limit effort="100.0" lower="-0.24" upper="0.24" velocity="100.0"/>
+    <dynamics friction="1.0" damping="0.1"/>
   </joint>
   <xacro:rocker_link name="R"/>
@@ -102,6 +102,6 @@
     <child link="rocker_R_link"/>
     <axis xyz="0 1 0"/>
-    <limit effort="10" lower="-0.24" upper="0.24" velocity="0.5"/>
-    <dynamics friction="0.1" damping="0.1"/>
+    <limit effort="100.0" lower="-0.24" upper="0.24" velocity="100.0"/>
+    <dynamics friction="1.0" damping="0.1"/>
     <mimic joint="rocker_L_joint"/>
   </joint>
@@ -112,4 +112,6 @@
     <child link="wheel_FL_link"/>
     <axis xyz="0 -1 0"/>
+    <limit effort="2.0" velocity="6.0"/>
+    <dynamics friction="0.3125" damping="0.1"/>
   </joint>
   <xacro:wheel_link name="RL" model="A"/>
@@ -119,4 +121,6 @@
     <child link="wheel_RL_link"/>
     <axis xyz="0 -1 0"/>
+    <limit effort="2.0" velocity="6.0"/>
+    <dynamics friction="0.3125" damping="0.1"/>
   </joint>
   <xacro:wheel_link name="FR" model="B"/>
@@ -126,4 +130,6 @@
     <child link="wheel_FR_link"/>
     <axis xyz="0 1 0"/>
+    <limit effort="2.0" velocity="6.0"/>
+    <dynamics friction="0.3125" damping="0.1"/>
   </joint>
   <xacro:wheel_link name="RR" model="B"/>
@@ -133,4 +139,6 @@
     <child link="wheel_RR_link"/>
     <axis xyz="0 1 0"/>
+    <limit effort="2.0" velocity="6.0"/>
+    <dynamics friction="0.3125" damping="0.1"/>
   </joint>
   <xacro:if value="$(arg default_antenna)">
